Commit message: Update ares8_rover.urdf

File: ares8_rover_description/urdf/ares8_rover.urdf (robot description, URDF)
Before this commit: robot ares8_rover, 9 links, 8 joints
Links:
- link base_link: geometry collision mesh filename=file:///home/karisora/ros2_ws/src/ares8_rover_description/m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 scale=0.001 0.001 0.001; visual mesh filename=file:///home/karisora/ros2_ws/src/ares8_rover_description/m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 scale=0.001 0.001 0.001
- link steering_link_lb_1: geometry collision mesh filename=file:///home/karisora/ros2_ws/src/ares8_rover_description/m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 scale=0.001 0.001 0.001; visual mesh filename=file:///home/karisora/ros2_ws/src/ares8_rover_description/m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 scale=0.001 0.001 0.001
- link steering_link_lf_1: geometry collision mesh filename=file:///home/karisora/ros2_ws/src/ares8_rover_description/m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 scale=0.001 0.001 0.001; visual mesh filename=file:///home/karisora/ros2_ws/src/ares8_rover_description/m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 scale=0.001 0.001 0.001
- link steering_link_rb_1: geometry collision mesh filename=file:///home/karisora/ros2_ws/src/ares8_rover_description/m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 scale=0.001 0.001 0.001; visual mesh filename=file:///home/karisora/ros2_ws/src/ares8_rover_description/m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 scale=0.001 0.001 0.001
- link steering_link_rf_1: geometry collision mesh filename=file:///home/karisora/ros2_ws/src/ares8_rover_description/m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 scale=0.001 0.001 0.001; visual mesh filename=file:///home/karisora/ros2_ws/src/ares8_rover_description/m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 scale=0.001 0.001 0.001
- link tire_LB_link_1: geometry collision mesh filename=file:///home/karisora/ros2_ws/src/ares8_rover_description/m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 scale=0.001 0.001 0.001; visual mesh filename=file:///home/karisora/ros2_ws/src/ares8_rover_description/m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 scale=0.001 0.001 0.001
- link tire_LF_link_1: geometry collision mesh filename=file:///home/karisora/ros2_ws/src/ares8_rover_description/m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 scale=0.001 0.001 0.001; visual mesh filename=file:///home/karisora/ros2_ws/src/ares8_rover_description/m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 scale=0.001 0.001 0.001
- link tire_RB_link_1: geometry collision mesh filename=file:///home/karisora/ros2_ws/src/ares8_rover_description/m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 scale=0.001 0.001 0.001; visual mesh filename=file:///home/karisora/ros2_ws/src/ares8_rover_description/m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 scale=0.001 0.001 0.001
- link tire_RF_link_1: geometry collision mesh filename=file:///home/karisora/ros2_ws/src/ares8_rover_description/m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 scale=0.001 0.001 0.001; visual mesh filename=file:///home/karisora/ros2_ws/src/ares8_rover_description/m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 scale=0.001 0.001 0.001
